File: src/icedev.kicad_sch (KiCad schematic)
At the start: 52 parts, among them J1 Conn_01x08, J11 USB_C_Receptacle_PowerOnly_6P, J2 Conn_02x01, J3 Conn_01x16, J4 Conn_02x01, J5 Conn_02x01, J6 Conn_01x16, J7 Conn_02x02_Odd_Even, J8 Conn_01x03, J9 Conn_02x01, U1 ICE40UP5K-SG48ITR, U2 AMS1117-1.2, U3 AMS1117-3.3, U4 W25Q128JVS, U5 FM24C64B, X1 MPUOSC

Commit message: Rev 2
Parts:
- removed J3, J6: Conn_01x16, Connector_PinHeader_2.54mm:PinHeader_1x16_P2.54mm_Vertical, symbol Connector_Generic:Conn_01x16
- added C23, C24: 0.1u, Capacitor_SMD:C_0402_1005Metric, symbol Device:C
- added J10, J12: Conn_01x18, Connector_PinSocket_2.54mm:PinSocket_1x18_P2.54mm_Vertical, symbol Connector_Generic:Conn_01x18
- added J3: USB_C_Receptacle_USB2.0_14P, Connector_USB:USB_C_Receptacle_GCT_USB4105-xx-A_16P_TopMnt_Horizontal, symbol Connector:USB_C_Receptacle_USB2.0_14P
- added R26, R27: 5.1K, Resistor_SMD:R_0805_2012Metric_Pad1.20x1.40mm_HandSolder, symbol Device:R
- D1: value MBR130 -> Schottky Diode; JLCPCB Part # C48974 -> C8598
- J1: footprint Connector_PinHeader_2.54mm:PinHeader_1x08_P2.54mm_Vertical -> Connector_PinSocket_2.54mm:PinSocket_1x08_P2.54mm_Vertical
Connections:
- net +5V: now also C23.1, C24.1, J10.2 (Pin_2), J3.A4 (VBUS), J3.A9 (VBUS), J3.B4 (VBUS), J3.B9 (VBUS)
- net CLK: now also J12.5 (Pin_5)
- net GND: now also J11.S1 (SHIELD), C23.2, C24.2, J10.1 (Pin_1), J12.1 (Pin_1), J12.2 (Pin_2), J3.A1 (GND), J3.A12 (GND), J3.B1 (GND), J3.B12 (GND), J3.S1 (SHIELD), R26.2, R27.1
- net IO13: now also J12.11 (Pin_11)
- net IO16: now also J12.12 (Pin_12)
- net IO18: now also J12.13 (Pin_13)
- net IO20: now also J12.14 (Pin_14)
- net IO22: now also J12.15 (Pin_15)
- net IO23: now also J12.16 (Pin_16)
- net IO24: now also J12.17 (Pin_17)
- net IO25: now also J12.18 (Pin_18)
- net IO29: now also J10.18 (Pin_18)
- net IO31: now also J10.17 (Pin_17)
- net IO36: now also J10.16 (Pin_16)
- net IO37: now also J10.15 (Pin_15)
- net IO38: now also J10.14 (Pin_14)
- net IO39: now also J10.13 (Pin_13)
- net IO4: now also J12.6 (Pin_6)
- net IO41: now also J10.12 (Pin_12)
- net IO42: now also J10.11 (Pin_11)
- net IO43: now also J10.10 (Pin_10)
- net IO44: now also J10.9 (Pin_9)
- net IO45: now also J10.8 (Pin_8)
- net IO46: now also J10.7 (Pin_7)
- net IO48: now also J10.6 (Pin_6)
- net IO49: now also J10.5 (Pin_5)
- net IO5: now also J12.7 (Pin_7)
- net IO50: now also J10.4 (Pin_4)
- net IO51: now also J10.3 (Pin_3)
- net IO6: now also J12.8 (Pin_8)
- net IO8: now also J12.9 (Pin_9)
- net IO9: now also J12.10 (Pin_10)
- net IO0 renamed D-
- net D-: now also J12.3 (Pin_3), J3.A7 (D-), J3.B7 (D-)
- net IO2 renamed D+
- net D+: now also J12.4 (Pin_4), J3.A6 (D+), J3.B6 (D+)
- new net: J3.B5 (CC2), R27.2
- new net: J3.A5 (CC1), R26.1
Other:
- company: (none) -> Cyao
- title: (none) -> Icedev
- moved on the sheet: C10, C16, C20, C4, C8, C9, D1, J11, R20, R21, U1D

Commit message: Some more improvements and readme images
Parts:
- removed C1, C10, C2, C3, C4, C8: 0.1u, Capacitor_SMD:C_0402_1005Metric, symbol Device:C
- removed C5, C6, C7, C9: 10n, Capacitor_SMD:C_0402_1005Metric, symbol Device:C
- removed D1: Schottky Diode, Diode_SMD:D_SOD-123, symbol Device:D
- removed D2, D4: G, LED_SMD:LED_0805_2012Metric, symbol Device:LED
- removed D3: R, LED_SMD:LED_0603_1608Metric, symbol Device:LED
- removed D5: B, LED_SMD:LED_0201_0603Metric_Pad0.64x0.40mm_HandSolder, symbol Device:LED
- removed J1: Conn_01x08, Connector_PinSocket_2.54mm:PinSocket_1x08_P2.54mm_Vertical, symbol Connector_Generic:Conn_01x08
- removed J10, J12: Conn_01x18, Connector_PinSocket_2.54mm:PinSocket_1x18_P2.54mm_Vertical, symbol Connector_Generic:Conn_01x18
- removed J2, J4: Conn_02x01, Connector_PinHeader_2.54mm:PinHeader_2x01_P2.54mm_Vertical, symbol Connector_Generic:Conn_02x01
- removed J8: Conn_01x03, Connector_PinHeader_2.54mm:PinHeader_1x03_P2.54mm_Vertical, symbol Connector_Generic:Conn_01x03
- removed R19, R22, R23, R24, R25: 1K, Resistor_SMD:R_0805_2012Metric, symbol Device:R
- removed U1: ICE40UP5K-SG48ITR, Package_DFN_QFN:QFN-48-1EP_7x7mm_P0.5mm_EP5.6x5.6mm, symbol FPGA_Lattice:ICE40UP5K-SG48ITR
- added H1, H2: MountingHole, MountingHole:MountingHole_2.2mm_M2, symbol Mechanical:MountingHole
- J11, J3, J5, J7, J9: now fitted
- R20, R21: footprint Resistor_SMD:R_0805_2012Metric_Pad1.20x1.40mm_HandSolder -> Resistor_SMD:R_0402_1005Metric; JLCPCB Part # (none) -> C25905; now fitted
- R26, R27: footprint Resistor_SMD:R_0805_2012Metric_Pad1.20x1.40mm_HandSolder -> Resistor_SMD:R_0805_2012Metric; JLCPCB Part # (none) -> C27834; now fitted
- X1: JLCPCB Part # C9006 -> C13738
Other:
- added sheet ice40 (ice40.kicad_sch)
- added sheet io (io.kicad_sch)
- note added: "128MiB NOR flash"
- note added: "16MHz Crystal"
- note added: "64kb EEPROM"
- note added: "LDO Regulators"
- note added: "USB connectors"
- moved on the sheet: C12, C13, C14, C15, C16, C17, C18, C19, C20, C21, C23, C24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

Commit message: Off to prod!
Parts:
- added U6: SRV05-4, PCM_marbastlib-various:SOT-23-6-routable, symbol PCM_marbastlib-various:SRV05-4
- H1, H2, J11, J3, J5, J7, J9: now not fitted
Connections:
- net +5V: now also U6.5 (VP)
- net D+: now also U6.6 (IO4)
- net D-: now also U6.1 (IO1)
- net GND: now also U6.2 (VN)
Other:
- note added: "For programming Flash"
- note added: "For programming iCE"
- note added: "For programming iCE cut traces connecting J15 and J16 pads. Short the pads 1 and 2 together of the J15 and J16 respectively. For programming Flash reverse the operations. Credits: ICEBreake"
- note added: "J18: Remove jumper when only programming iCE Replace jumper for programming Flash and for normal operation"
- moved on the sheet: U5
