File: src/io.kicad_sch (KiCad schematic)
At the start: 3 parts, among them J1 Conn_01x08, J10 Conn_01x18, J12 Conn_01x18

Commit message: Off to prod!
Parts:
- J1, J10, J12: now not fitted
Changed lines of the file:
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@@
 		(in_bom yes)
 		(on_board yes)
-		(dnp no)
+		(dnp yes)
 		(property "Reference" "J1"
 			(at 104.14 123.19 0)
@@
 		(in_bom yes)
 		(on_board yes)
-		(dnp no)
+		(dnp yes)
 		(property "Reference" "J10"
 			(at 115.57 53.34 0)
@@
 		(in_bom yes)
 		(on_board yes)
-		(dnp no)
+		(dnp yes)
 		(property "Reference" "J12"
 			(at 102.87 53.34 0)
